Commit message: added second camera2

File: robbie/urdf/robbie.xacro (robot description, xacro)
@@ -105,4 +105,18 @@
     </visual>
   </link>
+  <link name='camera2_link'>
+    <xacro:box_inertial name="camera2_link" m="${camera_mass}" x="${camera_width}" y="${camera_length}" z="${camera_height}"/>
+    <collision name='camera2_link_collision'>
+      <geometry>
+        <box size="${camera_length} ${camera_width} ${camera_height}"/>
+      </geometry>
+    </collision>
+    <visual name='camera2_link_visual'>
+      <origin xyz="0 0 0" rpy=" 0 0 0"/>
+      <geometry>
+        <box size="${camera_length} ${camera_width} ${camera_height}"/>
+      </geometry>
+    </visual>
+  </link>
   <joint name="wheel_FR_joint" type="continuous">
     <parent link="chassis"/>
@@ -138,4 +152,9 @@
     <origin xyz="${chassis_length/2} 0 ${chassis_height/2+camera_height/2}"/>
   </joint>
+  <joint name="camera2_joint" type="fixed">
+    <parent link="chassis"/>
+    <child link="camera2_link"/>
+    <origin xyz="${chassis_length/2} 0 ${chassis_height/2+camera_height*1.5}"/>
+  </joint>
   <gazebo reference="chassis">
     <material>Gazebo/Orange</material>
@@ -157,56 +176,41 @@
   </gazebo>
   <gazebo>
-    <plugin name="skid_steer_drive_controller" filename="libgazebo_ros_skid_steer_drive.so">
-      <updateRate>100.0</updateRate>
-      <leftFrontJoint>wheel_FL_joint</leftFrontJoint>
-      <rightFrontJoint>wheel_FR_joint</rightFrontJoint>
-      <leftRearJoint>wheel_RL_joint</leftRearJoint>
-      <rightRearJoint>wheel_RR_joint</rightRearJoint>
-      <wheelSeparation>0.4</wheelSeparation>
-      <wheelDiameter>0.215</wheelDiameter>
-      <robotBaseFrame>base_link</robotBaseFrame>
-      <torque>20</torque>
-      <topicName>cmd_vel</topicName>
-      <broadcastTF>false</broadcastTF>
+    <plugin name="skid_steer_drive" filename="libgazebo_ros_skid_steer_drive.so">
+      <ros>
+        <namespace>/robot</namespace>
+        <param name="left_wheel_joint">wheel_FL_joint</param>
+        <param name="right_wheel_joint">wheel_FR_joint</param>
+      </ros>
     </plugin>
   </gazebo>
-  <gazebo reference="camera_link">
-    <sensor type="camera" name="camera1">
-      <update_rate>30.0</update_rate>
-      <camera name="head">
-        <horizontal_fov>1.3962634</horizontal_fov>
-        <image>
-          <width>800</width>
-          <height>800</height>
-          <format>R8G8B8</format>
-        </image>
-        <clip>
-          <near>0.02</near>
-          <far>300</far>
-        </clip>
-        <noise>
-          <type>gaussian</type>
-          <!-- Noise is sampled independently per pixel on each frame.
-              That pixel's noise value is added to each of its color
-              channels, which at that point lie in the range [0,1]. -->
-          <mean>0.0</mean>
-          <stddev>0.007</stddev>
-        </noise>
+  <gazebo>
+    <plugin name="camera_plugin" filename="libgazebo_ros_camera.so">
+      <ros>
+        <namespace>/robot</namespace>
+        <param name="camera_name">camera1</param>
+      </ros>
+      <camera name="camera1">
+        <horizontal_fov>1.396</horizontal_fov>
+        <image_width>640</image_width>
+        <image_height>480</image_height>
+        <update_rate>30</update_rate>
+        <format>R8G8B8</format>
       </camera>
-      <plugin name="camera_controller" filename="libgazebo_ros_camera.so">
-        <alwaysOn>true</alwaysOn>
-        <updateRate>0.0</updateRate>
-        <cameraName>rrbot/camera1</cameraName>
-        <imageTopicName>image_raw</imageTopicName>
-        <cameraInfoTopicName>camera_info</cameraInfoTopicName>
-        <frameName>camera_link</frameName>
-        <hackBaseline>0.07</hackBaseline>
-        <distortionK1>0.0</distortionK1>
-        <distortionK2>0.0</distortionK2>
-        <distortionK3>0.0</distortionK3>
-        <distortionT1>0.0</distortionT1>
-        <distortionT2>0.0</distortionT2>
-      </plugin>
-    </sensor>
+    </plugin>
+  </gazebo>
+  <gazebo>
+    <plugin name="camera2_plugin" filename="libgazebo_ros_camera.so">
+      <ros>
+        <namespace>/robot</namespace>
+        <param name="camera_name">camera2</param>
+      </ros>
+      <camera name="camera2">
+        <horizontal_fov>1.396</horizontal_fov>
+        <image_width>640</image_width>
+        <image_height>480</image_height>
+        <update_rate>30</update_rate>
+        <format>R8G8B8</format>
+      </camera>
+    </plugin>
   </gazebo>
 </robot>

Commit message: camera2 and camera3

File: robbie/urdf/robbie.xacro (robot description, xacro)
@@ -119,4 +119,18 @@
     </visual>
   </link>
+    <link name='camera3_link'>
+    <xacro:box_inertial name="camera3_link" m="${camera_mass}" x="${camera_width}" y="${camera_length}" z="${camera_height}"/>
+    <collision name='camera3_link_collision'>
+      <geometry>
+        <box size="${camera_length} ${camera_width} ${camera_height}"/>
+      </geometry>
+    </collision>
+    <visual name='camera3_link_visual'>
+      <origin xyz="0 0 0" rpy=" 0 0 0"/>
+      <geometry>
+        <box size="${camera_length} ${camera_width} ${camera_height}"/>
+      </geometry>
+    </visual>
+  </link>
   <joint name="wheel_FR_joint" type="continuous">
     <parent link="chassis"/>
@@ -155,5 +169,10 @@
     <parent link="chassis"/>
     <child link="camera2_link"/>
-    <origin xyz="${chassis_length/2} 0 ${chassis_height/2+camera_height*1.5}"/>
+    <origin xyz="${chassis_length/2} ${chassis_width/2} ${chassis_height/2 + camera_height/2}" rpy="0 0 0.7854"/>
+  </joint>
+    <joint name="camera3_joint" type="fixed">
+    <parent link="chassis"/>
+    <child link="camera3_link"/>
+    <origin xyz="${chassis_length/2} -${chassis_width/2} ${chassis_height/2 + camera_height/2}" rpy="0 0 -0.7854"/>
   </joint>
   <gazebo reference="chassis">
@@ -163,4 +182,10 @@
     <material>Gazebo/Blue</material>
   </gazebo>
+  <gazebo reference="camera2_link">
+    <material>Gazebo/Blue</material>
+  </gazebo>
+  <gazebo reference="camera3_link">
+    <material>Gazebo/Blue</material>
+  </gazebo>
   <gazebo reference="wheel_FL">
     <material>Gazebo/Yellow</material>
@@ -176,41 +201,128 @@
   </gazebo>
   <gazebo>
-    <plugin name="skid_steer_drive" filename="libgazebo_ros_skid_steer_drive.so">
-      <ros>
-        <namespace>/robot</namespace>
-        <param name="left_wheel_joint">wheel_FL_joint</param>
-        <param name="right_wheel_joint">wheel_FR_joint</param>
-      </ros>
+    <plugin name="skid_steer_drive_controller" filename="libgazebo_ros_skid_steer_drive.so">
+      <updateRate>100.0</updateRate>
+      <leftFrontJoint>wheel_FL_joint</leftFrontJoint>
+      <rightFrontJoint>wheel_FR_joint</rightFrontJoint>
+      <leftRearJoint>wheel_RL_joint</leftRearJoint>
+      <rightRearJoint>wheel_RR_joint</rightRearJoint>
+      <wheelSeparation>0.4</wheelSeparation>
+      <wheelDiameter>0.215</wheelDiameter>
+      <robotBaseFrame>base_link</robotBaseFrame>
+      <torque>20</torque>
+      <topicName>cmd_vel</topicName>
+      <broadcastTF>false</broadcastTF>
     </plugin>
   </gazebo>
-  <gazebo>
-    <plugin name="camera_plugin" filename="libgazebo_ros_camera.so">
-      <ros>
-        <namespace>/robot</namespace>
-        <param name="camera_name">camera1</param>
-      </ros>
-      <camera name="camera1">
-        <horizontal_fov>1.396</horizontal_fov>
-        <image_width>640</image_width>
-        <image_height>480</image_height>
-        <update_rate>30</update_rate>
-        <format>R8G8B8</format>
+  <gazebo reference="camera_link">
+    <sensor type="camera" name="camera1">
+      <update_rate>30.0</update_rate>
+      <camera name="head">
+        <horizontal_fov>1.3962634</horizontal_fov>
+        <image>
+          <width>800</width>
+          <height>800</height>
+          <format>R8G8B8</format>
+        </image>
+        <clip>
+          <near>0.02</near>
+          <far>300</far>
+        </clip>
+        <noise>
+          <type>gaussian</type>
+          <!-- Noise is sampled independently per pixel on each frame.
+              That pixel's noise value is added to each of its color
+              channels, which at that point lie in the range [0,1]. -->
+          <mean>0.0</mean>
+          <stddev>0.007</stddev>
+        </noise>
       </camera>
-    </plugin>
-  </gazebo>
-  <gazebo>
-    <plugin name="camera2_plugin" filename="libgazebo_ros_camera.so">
-      <ros>
-        <namespace>/robot</namespace>
-        <param name="camera_name">camera2</param>
-      </ros>
-      <camera name="camera2">
-        <horizontal_fov>1.396</horizontal_fov>
-        <image_width>640</image_width>
-        <image_height>480</image_height>
-        <update_rate>30</update_rate>
-        <format>R8G8B8</format>
-      </camera>
-    </plugin>
-  </gazebo>
+      <plugin name="camera_controller" filename="libgazebo_ros_camera.so">
+        <alwaysOn>true</alwaysOn>
+        <updateRate>0.0</updateRate>
+        <cameraName>rrbot/camera1</cameraName>
+        <imageTopicName>image_raw</imageTopicName>
+        <cameraInfoTopicName>camera_info</cameraInfoTopicName>
+        <frameName>camera_link</frameName>
+        <hackBaseline>0.07</hackBaseline>
+        <distortionK1>0.0</distortionK1>
+        <distortionK2>0.0</distortionK2>
+        <distortionK3>0.0</distortionK3>
+        <distortionT1>0.0</distortionT1>
+        <distortionT2>0.0</distortionT2>
+      </plugin>
+    </sensor>
+  </gazebo>
+  <gazebo reference="camera2_link">
+    <sensor type="camera" name="camera2">
+        <update_rate>30.0</update_rate>
+        <camera name="camera2">
+            <horizontal_fov>1.3962634</horizontal_fov>
+            <image>
+                <width>800</width>
+                <height>800</height>
+                <format>R8G8B8</format>
+            </image>
+            <clip>
+                <near>0.02</near>
+                <far>300</far>
+            </clip>
+            <noise>
+                <type>gaussian</type>
+                <mean>0.0</mean>
+                <stddev>0.007</stddev>
+            </noise>
+        </camera>
+        <plugin name="camera2_controller" filename="libgazebo_ros_camera.so">
+            <alwaysOn>true</alwaysOn>
+            <updateRate>0.0</updateRate>
+            <cameraName>rrbot/camera2</cameraName>
+            <imageTopicName>image_raw</imageTopicName>
+            <cameraInfoTopicName>camera_info</cameraInfoTopicName>
+            <frameName>camera2_link</frameName>
+            <hackBaseline>0.07</hackBaseline>
+            <distortionK1>0.0</distortionK1>
+            <distortionK2>0.0</distortionK2>
+            <distortionK3>0.0</distortionK3>
+            <distortionT1>0.0</distortionT1>
+            <distortionT2>0.0</distortionT2>
+        </plugin>
+    </sensor>
+</gazebo>
+<gazebo reference="camera3_link">
+    <sensor type="camera" name="camera3">
+        <update_rate>30.0</update_rate>
+        <camera name="camera3">
+            <horizontal_fov>1.3962634</horizontal_fov>
+            <image>
+                <width>800</width>
+                <height>800</height>
+                <format>R8G8B8</format>
+            </image>
+            <clip>
+                <near>0.02</near>
+                <far>300</far>
+            </clip>
+            <noise>
+                <type>gaussian</type>
+                <mean>0.0</mean>
+                <stddev>0.007</stddev>
+            </noise>
+        </camera>
+        <plugin name="camera3_controller" filename="libgazebo_ros_camera.so">
+            <alwaysOn>true</alwaysOn>
+            <updateRate>0.0</updateRate>
+            <cameraName>rrbot/camera3</cameraName>
+            <imageTopicName>image_raw</imageTopicName>
+            <cameraInfoTopicName>camera_info</cameraInfoTopicName>
+            <frameName>camera3_link</frameName>
+            <hackBaseline>0.07</hackBaseline>
+            <distortionK1>0.0</distortionK1>
+            <distortionK2>0.0</distortionK2>
+            <distortionK3>0.0</distortionK3>
+            <distortionT1>0.0</distortionT1>
+            <distortionT2>0.0</distortionT2>
+        </plugin>
+    </sensor>
+</gazebo>
 </robot>
